File: ecad/_autosave-barometer-deck.kicad_pcb (KiCad board)
At the start: 2 copper layers, 25.2 x 27.3 mm, 5 parts, among them IC1 BMP390, P1 CF_EXP_LEFT, P2 CF_EXP_RIGHT, U1 NINA-W106-10B

Commit message: jtag support
Parts:
- added C1: 1u, Capacitor_SMD:C_0402_1005Metric, F.Cu at (101.1, 96.2)
- added C2: 100n, Capacitor_SMD:C_0402_1005Metric, F.Cu at (101.1, 98.2)
- added C3: 10u, Capacitor_SMD:C_0402_1005Metric, F.Cu at (101.1, 100.1)
- added C4: 100n, Capacitor_SMD:C_0402_1005Metric, F.Cu at (101.1, 102.1)
- added C5: 100n, Capacitor_SMD:C_0402_1005Metric, F.Cu at (101.1, 104.1)
- added C6: 100n, Capacitor_SMD:C_0402_1005Metric, F.Cu at (101.1, 106.1)
- added C7: 100n, Capacitor_SMD:C_0402_1005Metric, F.Cu at (101.1, 108.0)
- added C8: 100n, Capacitor_SMD:C_0402_1005Metric, F.Cu at (101.1, 110.0)
- added D1: LED, LED_SMD:LED_0603_1608Metric, F.Cu at (107.5, 105.7)
- added D2: LED, LED_SMD:LED_0603_1608Metric, F.Cu at (107.5, 108.3)
- added IC1: MIC5353-3.3YMT-TR, MIC5353-3_3YMT-TR:SON50P160X160X60-7N-D, F.Cu at (111.5, 110.8)
- added J1: Conn_02x05_Odd_Even, Connector_PinHeader_1.27mm:PinHeader_2x05_P1.27mm_Horizontal, F.Cu at (148.7, 100.7)
- added R1: 4.7k, Resistor_SMD:R_0402_1005Metric, F.Cu at (104.0, 105.4)
- added R2: 4.7k, Resistor_SMD:R_0402_1005Metric, F.Cu at (104.0, 107.4)
- added R3: 10k, Resistor_SMD:R_0402_1005Metric, F.Cu at (104.0, 109.4)
- added R4: 1k, Resistor_SMD:R_0402_1005Metric, F.Cu at (104.0, 111.4)
- added R5: 1k, Resistor_SMD:R_0402_1005Metric, F.Cu at (104.0, 113.4)
- added U2: DS2431, Package_TO_SOT_SMD:SOT-23-3, F.Cu at (112.1, 106.6)
- P1, P2: footprint connectors:BF090-10-X-B2 -> Connector_PinSocket_2.00mm:PinSocket_1x10_P2.00mm_Vertical
- moved P1 9.28 mm to (148.3, 85.3), turned to -90 degrees
- moved P2 8.81 mm to (147.8, 109.0), turned to -90 degrees
- moved U1 3.07 mm to (148.1, 93.0)
- renumbered IC1 to IC2
Connections:
- IC2 pad 1: unconnected-(IC1-VDDIO-Pad1) -> +3.3V
- IC2 pad 10: unconnected-(IC1-VDD-Pad10) -> +3.3V
- IC2 pad 2: unconnected-(IC1-SCK-Pad2) -> SCK
- IC2 pad 3: unconnected-(IC1-VSS_1-Pad3) -> GND
- IC2 pad 4: unconnected-(IC1-SDI-Pad4) -> SDA
- IC2 pad 5: unconnected-(IC1-SDO-Pad5) -> +3.3V
- IC2 pad 6: unconnected-(IC1-CSB-Pad6) -> +3.3V
- IC2 pad 8: unconnected-(IC1-VSS_2-Pad8) -> GND
- IC2 pad 9: unconnected-(IC1-VSS_3-Pad9) -> GND
- P1 pad 10: unconnected-(P1-GND-Pad10) -> GND
- P2 pad 8: unconnected-(P2-OW-Pad8) -> OW
- P2 pad 9: unconnected-(P2-VCOM-Pad9) -> VCOM
- U1 pad 10: unconnected-(U1-VCC-Pad10) -> +3.3V
- U1 pad 12: unconnected-(U1-GND-Pad12) -> GND
- U1 pad 14: unconnected-(U1-GND-Pad14) -> GND
- U1 pad 19: unconnected-(U1-RESET_N-Pad19) -> RST
- U1 pad 21: unconnected-(U1-GPIO_21/UART_CTS/RMII_TXD0/SPI_V_MISO-Pad21) -> SDA
- U1 pad 22: unconnected-(U1-GPIO_22/UART_TXD-Pad22) -> TXD
- U1 pad 23: unconnected-(U1-GPIO_23/UART_RXD-Pad23) -> RXD
- U1 pad 24: unconnected-(U1-GPIO_24/RMII_MDIO-Pad24) -> SCK
- U1 pad 26: unconnected-(U1-GND-Pad26) -> GND
- U1 pad 27: unconnected-(U1-GPIO_27/RMII_CLK/SYS_BOOT-Pad27) -> BOOT
- U1 pad 30: unconnected-(U1-GND-Pad30) -> GND
- U1 pad 37: unconnected-(U1-GND-Pad37) -> GND
- U1 pad 38: unconnected-(U1-GND-Pad38) -> GND
- U1 pad 39: unconnected-(U1-GND-Pad39) -> GND
- U1 pad 40: unconnected-(U1-GND-Pad40) -> GND
- U1 pad 41: unconnected-(U1-GND-Pad41) -> GND
- U1 pad 42: unconnected-(U1-GND-Pad42) -> GND
- U1 pad 43: unconnected-(U1-GND-Pad43) -> GND
- U1 pad 44: unconnected-(U1-GND-Pad44) -> GND
- U1 pad 45: unconnected-(U1-GND-Pad45) -> GND
- U1 pad 46: unconnected-(U1-GND-Pad46) -> GND
- U1 pad 47: unconnected-(U1-GND-Pad47) -> GND
- U1 pad 48: unconnected-(U1-GND-Pad48) -> GND
- U1 pad 49: unconnected-(U1-GND-Pad49) -> GND
- U1 pad 5: unconnected-(U1-GPIO_5-Pad5) -> WIFI_LED
- U1 pad 50: unconnected-(U1-GND-Pad50) -> GND
- U1 pad 51: unconnected-(U1-GND-Pad51) -> GND
- U1 pad 52: unconnected-(U1-GND-Pad52) -> GND
- U1 pad 6: unconnected-(U1-GND-Pad6) -> GND
- U1 pad 9: unconnected-(U1-VCC_IO-Pad9) -> +3.3V
Other:
- board text removed: "uUSB TOP"
