File: ecad/barometer-deck.kicad_sch (KiCad schematic)
At the start: 24 parts, among them IC1 MIC5353-3.3YMT-TR, IC2 BMP390, J1 JTAG_EDGE, P1 CF_EXP_LEFT, P2 CF_EXP_RIGHT, U1 NINA-W106-10B, U2 DS2431

Commit message: layout done
Parts:
- removed C8: 100n, Capacitor_SMD:C_0402_1005Metric, symbol PutRocketLab_RCL:C_Small
- R4: renamed from R6; footprint (none) -> Resistor_SMD:R_0402_1005Metric
- renumbered R4 to R5, R5 to R6
Connections:
- net RXD: now also P1.2 (RX1)
- net TXD: now also P1.3 (TX1)
- net WIFI_LED: now also U1.29 (GPIO_29/SPI_V_CLK); no longer U1.5 (GPIO_5)
- net BOOT: no longer names the net of U1.27 (GPIO_27/RMII_CLK/SYS_BOOT)
- no-connect marks 17 -> 34

Commit message: project description
Other:
- company: Bitcraze AB -> michal es company
- title: Crazyflie 2.0 expansion boad template -> Barometer deck
Changed lines of the file:
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@@
 	(paper "A4")
 	(title_block
-		(title "Crazyflie 2.0 expansion boad template")
-		(date "20 okt 2014")
+		(title "Barometer deck")
+		(date "2026-10-30")
 		(rev "A")
-		(company "Bitcraze AB")
+		(company "michal es company")
 		(comment 1 "Licensed under CC-BY 4.0")
 	)
 	(rectangle
-		(start 11.684 12.954)
-		(end 73.66 63.5)
+		(start 12.954 12.954)
+		(end 74.93 63.5)
 		(stroke
 			(width 0)
